File: DAC_interface.kicad_sch (KiCad schematic)
At the start: 11 parts, among them IC2 ES9038Q2M, Y2 SiT8209AI-21-33S-100.000000X

Commit message: Adding logos and finish up bom
Parts:
- R2: Mouser Part Number 603-RT0805BRD0710KL -> 603-RC0805FR-7W10KL; Part Number RT0805BRD0710KL -> RC0805FR-7W10KL
Changed lines of the file:
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@@
       (effects (font (size 1.27 1.27)) hide)
     )
-    (property "Part Number" "RT0805BRD0710KL" (id 4) (at 181.61 104.14 0)
+    (property "Part Number" "RC0805FR-7W10KL" (id 4) (at 181.61 104.14 0)
       (effects (font (size 1.27 1.27)) hide)
     )
-    (property "Mouser Part Number" "603-RT0805BRD0710KL" (id 5) (at 181.61 104.14 0)
+    (property "Mouser Part Number" "603-RC0805FR-7W10KL" (id 5) (at 181.61 104.14 0)
       (effects (font (size 1.27 1.27)) hide)
     )
