File: power.kicad_sch (KiCad schematic)
At the start: 62 parts, among them IC10 TPS7A3001DGNT, IC11 ADP150AUJZ-3.3-R7, IC4 ADP150AUJZ-3.3-R7, IC5 ADP150AUJZ-3.3-R7, IC6 ADP150AUJZ-3.3-R7, IC7 ADP150AUJZ-3.3-R7, IC8 LT1026CS8#PBF, IC9 ADP7118ARDZ

Commit message: Adding more part numbers. WIP verifying part numbers
Parts:
- C50: Mouser Part Number (none) -> 80-C0805C104K8RAUTO; Part Number (none) -> C0805C104K8RACAUTO
- C71: Mouser Part Number (none) -> 963-LMK212ABJ106KG8T; Part Number (none) -> LMK212ABJ106KG8T
Changed lines of the file:
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@@
+      (effects (font (size 1.27 1.27)) hide)
+    )
+    (property "Part Number" "C0805C104K8RACAUTO" (id 4) (at 106.68 33.02 0)
+      (effects (font (size 1.27 1.27)) hide)
+    )
+    (property "Mouser Part Number" "80-C0805C104K8RAUTO" (id 5) (at 106.68 33.02 0)
       (effects (font (size 1.27 1.27)) hide)
     )
@@
       (effects (font (size 1.27 1.27)) hide)
     )
-    (property "Part Number" "" (id 4) (at 271.78 147.32 0)
-      (effects (font (size 1.27 1.27)) hide)
-    )
-    (property "Mouser Part Number" "" (id 5) (at 271.78 147.32 0)
-      (effects (font (size 1.27 1.27)) hide)
-    )
+    (property "Part Number" "LMK212ABJ106KG8T" (id 4) (at 271.78 147.32 0)
+      (effects (font (size 1.27 1.27)) hide)
+    )
+    (property "Mouser Part Number" "963-LMK212ABJ106KG8T" (id 5) (at 271.78 147.32 0)
+      (effects (font (size 1.27 1.27)) hide)
+    )

Commit message: Adding logos and finish up bom
Parts:
- IC11, IC4, IC5, IC6, IC7: Mouser Part Number N/A -> 584-ADP150AUJZ-3.3R7
Changed lines of the file:
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@@
       (effects (font (size 1.27 1.27)) (justify left) hide)
     )
-    (property "Mouser Part Number" "N/A" (id 8) (at 83.82 39.37 0)
+    (property "Mouser Part Number" "584-ADP150AUJZ-3.3R7" (id 8) (at 83.82 39.37 0)
       (effects (font (size 1.27 1.27)) (justify left) hide)
     )
@@
     (property "Arrow Price/Stock" "https://www.arrow.com/en/products/adp150aujz-3.3-r7/analog-devices?region=nac" (id 11) (at 83.82 46.99 0)
       (effects (font (size 1.27 1.27)) (justify left) hide)
+    )
+    (property "Part Number" "" (id 12) (at 59.69 26.67 0)
+      (effects (font (size 1.27 1.27)) hide)
     )
     (pin "1")
@@
       (effects (font (size 1.27 1.27)) (justify left) hide)
     )
-    (property "Mouser Part Number" "N/A" (id 8) (at 83.82 118.11 0)
+    (property "Mouser Part Number" "584-ADP150AUJZ-3.3R7" (id 8) (at 83.82 118.11 0)
       (effects (font (size 1.27 1.27)) (justify left) hide)
     )
@@
     (property "Arrow Price/Stock" "https://www.arrow.com/en/products/adp150aujz-3.3-r7/analog-devices?region=nac" (id 11) (at 83.82 125.73 0)
       (effects (font (size 1.27 1.27)) (justify left) hide)
+    )
+    (property "Part Number" "" (id 12) (at 59.69 105.41 0)
+      (effects (font (size 1.27 1.27)) hide)
     )
     (pin "1")
@@
       (effects (font (size 1.27 1.27)) (justify left) hide)
     )
-    (property "Mouser Part Number" "N/A" (id 8) (at 83.82 177.8 0)
+    (property "Mouser Part Number" "584-ADP150AUJZ-3.3R7" (id 8) (at 83.82 177.8 0)
       (effects (font (size 1.27 1.27)) (justify left) hide)
     )
@@
     (property "Arrow Price/Stock" "https://www.arrow.com/en/products/adp150aujz-3.3-r7/analog-devices?region=nac" (id 11) (at 83.82 185.42 0)
       (effects (font (size 1.27 1.27)) (justify left) hide)
+    )
+    (property "Part Number" "" (id 12) (at 59.69 165.1 0)
+      (effects (font (size 1.27 1.27)) hide)
     )
     (pin "1")
@@
       (effects (font (size 1.27 1.27)) (justify left) hide)
     )
-    (property "Mouser Part Number" "N/A" (id 8) (at 83.82 147.32 0)
+    (property "Mouser Part Number" "584-ADP150AUJZ-3.3R7" (id 8) (at 83.82 147.32 0)
       (effects (font (size 1.27 1.27)) (justify left) hide)
     )
@@
     (property "Arrow Price/Stock" "https://www.arrow.com/en/products/adp150aujz-3.3-r7/analog-devices?region=nac" (id 11) (at 83.82 154.94 0)
       (effects (font (size 1.27 1.27)) (justify left) hide)
+    )
+    (property "Part Number" "" (id 12) (at 59.69 134.62 0)
+      (effects (font (size 1.27 1.27)) hide)
     )
     (pin "1")
@@
       (effects (font (size 1.27 1.27)) (justify left) hide)
     )
-    (property "Mouser Part Number" "N/A" (id 8) (at 83.82 73.66 0)
+    (property "Mouser Part Number" "584-ADP150AUJZ-3.3R7" (id 8) (at 83.82 73.66 0)
       (effects (font (size 1.27 1.27)) (justify left) hide)
     )
@@
       (effects (font (size 1.27 1.27)) (justify left) hide)
     )
-    (pin "1")
+    (property "Part Number" "" (id 12) (at 59.69 60.96 0)
+      (effects (font (size 1.27 1.27)) hide)
+    )
+    (pin "1")

Commit message: Adding readme
Parts:
- C45, C46, C47: value 47u_16V -> 47u
Changed lines of the file:
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@@
       (effects (font (size 1.27 1.27)) (justify left))
     )
-    (property "Value" "47u_16V" (id 1) (at 99.06 112.3949 0)
+    (property "Value" "47u" (id 1) (at 99.06 112.3949 0)
       (effects (font (size 1.27 1.27)) (justify left))
     )
@@
       (effects (font (size 1.27 1.27)) (justify left))
     )
-    (property "Value" "47u_16V" (id 1) (at 99.06 141.6049 0)
+    (property "Value" "47u" (id 1) (at 99.06 141.6049 0)
       (effects (font (size 1.27 1.27)) (justify left))
     )
@@
       (effects (font (size 1.27 1.27)) (justify left))
     )
-    (property "Value" "47u_16V" (id 1) (at 99.06 172.0849 0)
-      (effects (font (size 1.27 1.27)) (justify left))
-    )
+    (property "Value" "47u" (id 1) (at 99.06 172.0849 0)
+      (effects (font (size 1.27 1.27)) (justify left))
+    )
