File: KiCAD/DAC_interface.kicad_sch (KiCad schematic)
At the start: 11 parts, among them IC2 ES9038Q2M, Y2 SiT8209AI-21-33S-100.000000X

Commit message: Reorganzing
Parts:
- C2, C5: Mouser Part Number 581-0805YC224JAT2A -> 187-CL21B224KAFNNNG; Part Number 0805YC224JAT2A -> CL21B224KAFNNNG
Changed lines of the file:
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@@
       (effects (font (size 1.27 1.27)) hide)
     )
-    (property "Part Number" "0805YC224JAT2A" (id 4) (at 246.38 81.28 0)
+    (property "Part Number" "CL21B224KAFNNNG" (id 4) (at 246.38 81.28 0)
       (effects (font (size 1.27 1.27)) hide)
     )
-    (property "Mouser Part Number" "581-0805YC224JAT2A" (id 5) (at 246.38 81.28 0)
+    (property "Mouser Part Number" "187-CL21B224KAFNNNG" (id 5) (at 246.38 81.28 0)
       (effects (font (size 1.27 1.27)) hide)
     )
@@
       (effects (font (size 1.27 1.27)) hide)
     )
-    (property "Part Number" "0805YC224JAT2A" (id 4) (at 52.07 88.9 0)
+    (property "Part Number" "CL21B224KAFNNNG" (id 4) (at 52.07 88.9 0)
       (effects (font (size 1.27 1.27)) hide)
     )
-    (property "Mouser Part Number" "581-0805YC224JAT2A" (id 5) (at 52.07 88.9 0)
+    (property "Mouser Part Number" "187-CL21B224KAFNNNG" (id 5) (at 52.07 88.9 0)
       (effects (font (size 1.27 1.27)) hide)
     )

Commit message: REV 1.0.1 does not work. Updating BOM IDs.
Parts:
- C3: Mouser Part Number 80-C0805C104K8RAUTO -> 603-CC805KKX5R7BB475; Part Number C0805C104K8RACAUTO -> CC0805KKX5R7BB475
Changed lines of the file:
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@@
       (effects (font (size 1.27 1.27)) hide)
     )
-    (property "Part Number" "C0805C104K8RACAUTO" (id 4) (at 59.69 88.9 0)
+    (property "Part Number" "CC0805KKX5R7BB475" (id 4) (at 59.69 88.9 0)
       (effects (font (size 1.27 1.27)) hide)
     )
-    (property "Mouser Part Number" "80-C0805C104K8RAUTO" (id 5) (at 59.69 88.9 0)
+    (property "Mouser Part Number" "603-CC805KKX5R7BB475" (id 5) (at 59.69 88.9 0)
       (effects (font (size 1.27 1.27)) hide)
     )

Commit message: Adding stuff for rev 2.0
Parts:
- C4: Mouser Part Number 581-0805ZD225KAT4A -> 963-TMK212B7225KGHT; Part Number 0805ZD225KAT4A -> TMK212B7225KGHT
Changed lines of the file:
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@@
       (effects (font (size 1.27 1.27)) hide)
     )
-    (property "Part Number" "0805ZD225KAT4A" (id 4) (at 181.61 118.11 0)
+    (property "Part Number" "TMK212B7225KGHT" (id 4) (at 181.61 118.11 0)
       (effects (font (size 1.27 1.27)) hide)
     )
-    (property "Mouser Part Number" "581-0805ZD225KAT4A" (id 5) (at 181.61 118.11 0)
+    (property "Mouser Part Number" "963-TMK212B7225KGHT" (id 5) (at 181.61 118.11 0)
       (effects (font (size 1.27 1.27)) hide)
     )
