File: KiCAD/output_stage.kicad_sch (KiCad schematic)
At the start: 41 parts, among them U2 OPA1612-Q1, U3 OPA1612-Q1, U4 OPA1622

Commit message: Reorganzing
Parts:
- C20, C21, C22, C23, C36, C37: Mouser Part Number 581-0805YC224JAT2A -> 187-CL21B224KAFNNNG; Part Number 0805YC224JAT2A -> CL21B224KAFNNNG
- R13, R15: Mouser Part Number 71-PNM0805E5001BST5 -> 652-CRT0805BY5001EAS; Part Number PNM0805E5001BST5 -> CRT0805-BY-5001EAS
- U2, U3: value OPA1612-Q1 -> OPA1612; Mouser Part Number 595-OPA1612AQDRQ1 -> 595-OPA1612AID; Part Number OPA1612AQDRQ1 -> OPA1612AID
Changed lines of the file:
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@@
       (effects (font (size 1.27 1.27)) hide)
     )
-    (property "Part Number" "0805YC224JAT2A" (id 4) (at 242.57 128.27 0)
-      (effects (font (size 1.27 1.27)) hide)
-    )
-    (property "Mouser Part Number" "581-0805YC224JAT2A" (id 5) (at 242.57 128.27 0)
+    (property "Part Number" "CL21B224KAFNNNG" (id 4) (at 242.57 128.27 0)
+      (effects (font (size 1.27 1.27)) hide)
+    )
+    (property "Mouser Part Number" "187-CL21B224KAFNNNG" (id 5) (at 242.57 128.27 0)
       (effects (font (size 1.27 1.27)) hide)
     )
@@
       (effects (font (size 1.27 1.27)) hide)
     )
-    (property "Part Number" "PNM0805E5001BST5" (id 4) (at 82.55 74.93 0)
-      (effects (font (size 1.27 1.27)) hide)
-    )
-    (property "Mouser Part Number" "71-PNM0805E5001BST5" (id 5) (at 82.55 74.93 0)
+    (property "Part Number" "CRT0805-BY-5001EAS" (id 4) (at 82.55 74.93 0)
+      (effects (font (size 1.27 1.27)) hide)
+    )
+    (property "Mouser Part Number" "652-CRT0805BY5001EAS" (id 5) (at 82.55 74.93 0)
       (effects (font (size 1.27 1.27)) hide)
     )
@@
       (effects (font (size 1.27 1.27)) hide)
     )
-    (property "Part Number" "0805YC224JAT2A" (id 4) (at 45.72 91.44 0)
-      (effects (font (size 1.27 1.27)) hide)
-    )
-    (property "Mouser Part Number" "581-0805YC224JAT2A" (id 5) (at 45.72 91.44 0)
+    (property "Part Number" "CL21B224KAFNNNG" (id 4) (at 45.72 91.44 0)
+      (effects (font (size 1.27 1.27)) hide)
+    )
+    (property "Mouser Part Number" "187-CL21B224KAFNNNG" (id 5) (at 45.72 91.44 0)
       (effects (font (size 1.27 1.27)) hide)
     )
@@
       (effects (font (size 1.27 1.27)) (justify left))
     )
-    (property "Value" "OPA1612-Q1" (id 1) (at 104.14 116.84 0)
+    (property "Value" "OPA1612" (id 1) (at 104.14 116.84 0)
       (effects (font (size 1.27 1.27)) (justify left))
     )
@@
       (effects (font (size 1.27 1.27)) hide)
     )
-    (property "Part Number" "OPA1612AQDRQ1" (id 4) (at 104.14 118.11 0)
-      (effects (font (size 1.27 1.27)) hide)
-    )
-    (property "Mouser Part Number" "595-OPA1612AQDRQ1" (id 5) (at 104.14 118.11 0)
+    (property "Part Number" "OPA1612AID" (id 4) (at 104.14 118.11 0)
+      (effects (font (size 1.27 1.27)) hide)
+    )
+    (property "Mouser Part Number" "595-OPA1612AID" (id 5) (at 104.14 118.11 0)
       (effects (font (size 1.27 1.27)) hide)
     )
@@
       (effects (font (size 1.27 1.27)) hide)
     )
-    (property "Part Number" "0805YC224JAT2A" (id 4) (at 45.72 113.03 0)
-      (effects (font (size 1.27 1.27)) hide)
-    )
-    (property "Mouser Part Number" "581-0805YC224JAT2A" (id 5) (at 45.72 113.03 0)
+    (property "Part Number" "CL21B224KAFNNNG" (id 4) (at 45.72 113.03 0)
+      (effects (font (size 1.27 1.27)) hide)
+    )
+    (property "Mouser Part Number" "187-CL21B224KAFNNNG" (id 5) (at 45.72 113.03 0)
       (effects (font (size 1.27 1.27)) hide)
     )
@@
       (effects (font (size 1.27 1.27)) hide)
     )
-    (property "Part Number" "0805YC224JAT2A" (id 4) (at 45.72 26.67 0)
-      (effects (font (size 1.27 1.27)) hide)
-    )
-    (property "Mouser Part Number" "581-0805YC224JAT2A" (id 5) (at 45.72 26.67 0)
+    (property "Part Number" "CL21B224KAFNNNG" (id 4) (at 45.72 26.67 0)
+      (effects (font (size 1.27 1.27)) hide)
+    )
+    (property "Mouser Part Number" "187-CL21B224KAFNNNG" (id 5) (at 45.72 26.67 0)
       (effects (font (size 1.27 1.27)) hide)
     )
@@
       (effects (font (size 1.27 1.27)) hide)
     )
-    (property "Part Number" "0805YC224JAT2A" (id 4) (at 45.72 177.8 0)
-      (effects (font (size 1.27 1.27)) hide)
-    )
-    (property "Mouser Part Number" "581-0805YC224JAT2A" (id 5) (at 45.72 177.8 0)
+    (property "Part Number" "CL21B224KAFNNNG" (id 4) (at 45.72 177.8 0)
+      (effects (font (size 1.27 1.27)) hide)
+    )
+    (property "Mouser Part Number" "187-CL21B224KAFNNNG" (id 5) (at 45.72 177.8 0)
       (effects (font (size 1.27 1.27)) hide)
     )
@@
       (effects (font (size 1.27 1.27)) hide)
     )
-    (property "Part Number" "PNM0805E5001BST5" (id 4) (at 82.55 161.29 0)
-      (effects (font (size 1.27 1.27)) hide)
-    )
-    (property "Mouser Part Number" "71-PNM0805E5001BST5" (id 5) (at 82.55 161.29 0)
+    (property "Part Number" "CRT0805-BY-5001EAS" (id 4) (at 82.55 161.29 0)
+      (effects (font (size 1.27 1.27)) hide)
+    )
+    (property "Mouser Part Number" "652-CRT0805BY5001EAS" (id 5) (at 82.55 161.29 0)
       (effects (font (size 1.27 1.27)) hide)
     )
@@
       (effects (font (size 1.27 1.27)) hide)
     )
-    (property "Part Number" "0805YC224JAT2A" (id 4) (at 242.57 30.48 0)
-      (effects (font (size 1.27 1.27)) hide)
-    )
-    (property "Mouser Part Number" "581-0805YC224JAT2A" (id 5) (at 242.57 30.48 0)
+    (property "Part Number" "CL21B224KAFNNNG" (id 4) (at 242.57 30.48 0)
+      (effects (font (size 1.27 1.27)) hide)
+    )
+    (property "Mouser Part Number" "187-CL21B224KAFNNNG" (id 5) (at 242.57 30.48 0)
       (effects (font (size 1.27 1.27)) hide)
     )
@@
       (effects (font (size 1.27 1.27)) (justify left))
     )
-    (property "Value" "OPA1612-Q1" (id 1) (at 104.14 30.48 0)
+    (property "Value" "OPA1612" (id 1) (at 104.14 30.48 0)
       (effects (font (size 1.27 1.27)) (justify left))
     )
@@
       (effects (font (size 1.27 1.27)) hide)
     )
-    (property "Part Number" "OPA1612AQDRQ1" (id 4) (at 104.14 31.75 0)
-      (effects (font (size 1.27 1.27)) hide)
-    )
-    (property "Mouser Part Number" "595-OPA1612AQDRQ1" (id 5) (at 104.14 31.75 0)
-      (effects (font (size 1.27 1.27)) hide)
-    )
+    (property "Part Number" "OPA1612AID" (id 4) (at 104.14 31.75 0)
+      (effects (font (size 1.27 1.27)) hide)
+    )
+    (property "Mouser Part Number" "595-OPA1612AID" (id 5) (at 104.14 31.75 0)
+      (effects (font (size 1.27 1.27)) hide)
+    )

Commit message: Adding stuff for rev 2.0
Parts:
- C24, C25: Mouser Part Number 581-0805ZD225KAT4A -> 963-TMK212B7225KGHT; Part Number 0805ZD225KAT4A -> TMK212B7225KGHT
Changed lines of the file:
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@@
       (effects (font (size 1.27 1.27)) hide)
     )
-    (property "Part Number" "0805ZD225KAT4A" (id 4) (at 88.9 161.29 0)
-      (effects (font (size 1.27 1.27)) hide)
-    )
-    (property "Mouser Part Number" "581-0805ZD225KAT4A" (id 5) (at 88.9 161.29 0)
+    (property "Part Number" "TMK212B7225KGHT" (id 4) (at 88.9 161.29 0)
+      (effects (font (size 1.27 1.27)) hide)
+    )
+    (property "Mouser Part Number" "963-TMK212B7225KGHT" (id 5) (at 88.9 161.29 0)
       (effects (font (size 1.27 1.27)) hide)
     )
@@
       (effects (font (size 1.27 1.27)) hide)
     )
-    (property "Part Number" "0805ZD225KAT4A" (id 4) (at 88.9 74.93 0)
-      (effects (font (size 1.27 1.27)) hide)
-    )
-    (property "Mouser Part Number" "581-0805ZD225KAT4A" (id 5) (at 88.9 74.93 0)
-      (effects (font (size 1.27 1.27)) hide)
-    )
+    (property "Part Number" "TMK212B7225KGHT" (id 4) (at 88.9 74.93 0)
+      (effects (font (size 1.27 1.27)) hide)
+    )
+    (property "Mouser Part Number" "963-TMK212B7225KGHT" (id 5) (at 88.9 74.93 0)
+      (effects (font (size 1.27 1.27)) hide)
+    )
