File: KiCAD/steDAC.kicad_pcb (KiCad board)
At the start: 2 copper layers, 100 x 80 mm, 157 parts, among them IC10 ADP7182ACPZN-R7, IC11 NCP161ASN330T1G, IC2 ES9038Q2M, IC3 ATSAMS70N20A-AN, IC4 NCP161ASN330T1G, IC5 NCP161ASN330T1G, IC6 NCP161ASN330T1G, IC7 NCP161ASN330T1G, IC8 LT1026CS8#PBF, IC9 ADP7118ARDZ, J2 USB4105-GF-A, J3 Conn_02x05_Odd_Even, J5 Conn_01x02, J6 Conn_01x04, J7 STX-3120-5B-284C, U2 OPA1612, U3 OPA1612, U4 OPA1622, Y2 SiT8209AI-21-33S-100.000000X, Y3 12MHz

Commit message: Adding stuff for rev 2.0
Parts:
- removed C70: 10u, Capacitor_SMD:C_0805_2012Metric_Pad1.18x1.45mm_HandSolder
- removed C77: 0.1u, Capacitor_SMD:C_0805_2012Metric_Pad1.18x1.45mm_HandSolder
- removed R31: 24k, Resistor_SMD:R_0805_2012Metric_Pad1.20x1.40mm_HandSolder
- added H2: MountingHole_Pad, MountingHole:MountingHole_2.2mm_M2_DIN965_Pad_TopBottom, F.Cu at (183.2, 58.9)
- added H3: MountingHole_Pad, MountingHole:MountingHole_2.2mm_M2_DIN965_Pad_TopBottom, F.Cu at (92.0, 59.8)
- added H4: MountingHole_Pad, MountingHole:MountingHole_2.2mm_M2_DIN965_Pad_TopBottom, F.Cu at (107.3, 122.4)
- added H5: MountingHole_Pad, MountingHole:MountingHole_2.2mm_M2_DIN965_Pad_TopBottom, F.Cu at (184.4, 130.2)
- added JP10: SolderJumper_2_Bridged, Jumper:SolderJumper-2_P1.3mm_Bridged2Bar_Pad1.0x1.5mm, B.Cu at (121.5, 110.1)
- added JP5: jumper, Jumper:SolderJumper-2_P1.3mm_Bridged2Bar_Pad1.0x1.5mm, B.Cu at (139.1, 90.6)
- added JP6: jumper, Jumper:SolderJumper-2_P1.3mm_Bridged2Bar_Pad1.0x1.5mm, B.Cu at (169.9, 89.6)
- added JP7: jumper, Jumper:SolderJumper-2_P1.3mm_Bridged2Bar_Pad1.0x1.5mm, B.Cu at (177.2, 89.6)
- added JP8: SolderJumper_2_Bridged, Jumper:SolderJumper-2_P1.3mm_Bridged2Bar_Pad1.0x1.5mm, B.Cu at (131.3, 90.7)
- added JP9: SolderJumper_2_Bridged, Jumper:SolderJumper-2_P1.3mm_Bridged2Bar_Pad1.0x1.5mm, B.Cu at (115.8, 110.1)
- C62: value 10u -> 4.7u
- C63: value 1n -> 2.2u
- C64: value 1u -> 10u; footprint Capacitor_THT:CP_Radial_D5.0mm_P2.00mm -> Capacitor_SMD:C_0805_2012Metric_Pad1.18x1.45mm_HandSolder
- C65: value 2.2u -> 4.7u; footprint Capacitor_THT:CP_Radial_D4.0mm_P1.50mm -> Capacitor_SMD:C_0805_2012Metric_Pad1.18x1.45mm_HandSolder
- C66: value 4.7u -> 10u
- C69: value 2.2u -> 47u; footprint Capacitor_THT:CP_Radial_D4.0mm_P1.50mm -> Capacitor_THT:CP_Radial_D5.0mm_P2.50mm
- IC8: value LT1026CS8#PBF -> MAX889SESA+; footprint SamacSys_Parts:SOIC127P599X175-8N -> SamacSys_Parts:SOIC127P600X175-8N
- IC9: value ADP7118ARDZ -> MAX38902AATA+T; footprint SamacSys_Parts:SOIC127P600X175-9N -> SamacSys_Parts:SON50P200X200X80-9N-D
- R11: value 1k -> 100k
- R30: value 10k -> 100k
- moved C63 40.6 mm to (109.3, 115.6), turned to -90 degrees
- moved C69 26.6 mm to (147.3, 81.1), turned to 90 degrees
- moved R30 24.3 mm to (120.6, 118.7), turned to 90 degrees
- moved R11 19.5 mm to (120.6, 114.6), turned to 90 degrees
- moved C65 18.2 mm to (132.8, 97.2)
- moved C66 7.12 mm to (107.8, 112.5), turned to 180 degrees
- moved FB3 6.49 mm to (136.3, 82.5), turned to 0 degrees
- moved C64 4.17 mm to (123.5, 116.7), turned to -90 degrees
- moved IC8 3.95 mm to (115.1, 114.4), turned to 0 degrees
- moved C62 3.51 mm to (133.1, 88.9)
- moved FB4 2.62 mm to (118.1, 65.7), turned to 180 degrees
- moved C68 2.44 mm to (136.0, 96.3), turned to 180 degrees
- moved IC9 1.51 mm to (134.6, 93.2), turned to -90 degrees
- moved C34 0.51 mm to (180.5, 130.2)
- moved R26 0.51 mm to (178.0, 130.2)
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Connections:
- C12 pad 2: +3V3 -> +1V2
- C58 pad 1: +3V3 -> +1V2
- C63 pad 2: GND -> Net-(C63-Pad2)
- C64 pad 2: Net-(C64-Pad2) -> GND
- C65 pad 1: GND -> +VDAC
- C65 pad 2: Net-(C65-Pad2) -> GNDREF
- C66 pad 1: GND -> DAC_5V
- C66 pad 2: DAC_5V -> GND
- C68 pad 1: Net-(C68-Pad1) -> +VDAC
- C68 pad 2: +VDAC -> Net-(C68-Pad2)
- C69 pad 1: +VDAC -> DAC_5V
- C69 pad 2: GNDREF -> GND
- C79 pad 2: +3V3 -> +1V2
- FB3 pad 1: +5V -> MCU_5V
- FB4 pad 1: +5V -> MCU_5V
- FB4 pad 2: MCU_5V -> Net-(JP3-Pad2)
- IC10 pad 3: Net-(C65-Pad2) -> Net-(IC10-Pad3)
- IC10 pad 6: Net-(C65-Pad2) -> Net-(C64-Pad1)
- IC11 pad 3: DAC_PWR_EN -> Net-(IC11-Pad3)
- IC3 pad 86: +3V3 -> +1V2
- IC3 pad 96: +3V3 -> +1V2
- IC6 pad 3: DAC_PWR_EN -> Net-(IC6-Pad3)
- IC7 pad 3: DAC_PWR_EN -> Net-(IC7-Pad3)
- IC8 pad 1: unconnected-(IC8-Pad1) -> DAC_5V
- IC8 pad 2: Net-(C64-Pad1) -> Net-(C63-Pad1)
- IC8 pad 3: Net-(C64-Pad2) -> GND
- IC8 pad 4: Net-(C65-Pad2) -> Net-(C63-Pad2)
- IC8 pad 5: GND -> Net-(C64-Pad1)
- IC8 pad 6: DAC_5V -> Net-(IC8-Pad6)
- IC8 pad 7: DAC_5V -> Net-(IC8-Pad7)
- IC8 pad 8: unconnected-(IC8-Pad8) -> GND
- IC9 pad 1: +VDAC -> DAC_5V
- IC9 pad 2: +VDAC -> GND
- IC9 pad 3: Net-(C68-Pad1) -> Net-(IC9-Pad3)
- IC9 pad 4: GNDREF -> DAC_5V
- IC9 pad 5: DAC_PWR_EN -> GNDREF
- IC9 pad 6: Net-(C63-Pad1) -> +VDAC
- IC9 pad 7: DAC_5V -> Net-(C68-Pad2)
- IC9 pad 8: DAC_5V -> +VDAC
- JP3 pad 2: +5V -> Net-(JP3-Pad2)
- R11 pad 1: Net-(C68-Pad1) -> Net-(C64-Pad1)
- R11 pad 2: Net-(C70-Pad1) -> Net-(IC8-Pad7)
- R30 pad 1: Net-(C68-Pad1) -> DAC_5V
- R30 pad 2: GNDREF -> Net-(C64-Pad1)
Routing:
- net +5V: track 36.8 -> 0.00 mm, vias 2 -> 0
- net MCU_5V: track 85.6 -> 112.1 mm, vias 2 -> 3
- net DAC_PWR_EN: track 74.0 -> 99.6 mm, vias 4 -> 3
- net Net-(C65-Pad2): track 19.1 -> 0.00 mm, vias 2 -> 0
- net Net-(C68-Pad1): track 17.1 -> 0.00 mm
- net +1V2: track 51.6 -> 68.2 mm
- net DAC_5V: track 139.4 -> 153.6 mm, vias 7 -> 6
- net +3V3: track 303.6 -> 292.7 mm, vias 14 -> 16
- net Net-(IC10-Pad3): track 0.00 -> 9.98 mm, vias 0 -> 1
- net Net-(IC8-Pad6): track 0.00 -> 7.69 mm, vias 0 -> 1
- net GND: track 36.0 -> 42.0 mm, vias 1 -> 4
- net Net-(C64-Pad1): track 6.02 -> 11.9 mm
- net Net-(C64-Pad2): track 5.72 -> 0.00 mm
- net Net-(IC9-Pad3): track 0.00 -> 5.30 mm, vias 0 -> 1
- net Net-(IC6-Pad3): track 0.00 -> 4.16 mm, vias 0 -> 1
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Other:
- board text added: "Rev 2.0"
- board text removed: "Rev 1.1.0"
